File: Electronics/Motherboard/CurrentVersion/Motherboard2.4 (small)/motherboard_2layers_v2.kicad_pcb (KiCad board)
At the start: 2 copper layers, 113.4 x 55.3 mm, 87 parts, among them J1 Conn_02x10_Odd_Even, J2 SSD1306, J3 USB_C_Receptacle_USB2.0_16P, J4 Micro_SD_Card_Det2, J5 Encoder, Q1 FDMS86202, Q2 FDMS86202, Q3 AO3400A, Q4 AO3400A, Q5 AO3400A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

Commit message: routed T0, T1, and T2. 30 more things to route but geez this is difficult
Routing:
- net T0: track 6.84 -> 68.7 mm, vias 0 -> 2
- net T1: track 6.68 -> 42.8 mm, vias 0 -> 4
- net T2: track 6.74 -> 34.7 mm, vias 0 -> 4
- net GND: track 394.8 -> 397.7 mm
- net +3V3: track 271.1 -> 272.2 mm
- net EN_E1: track 93.9 -> 94.7 mm
- net Net-(D3-DOUT): track 88.7 -> 89.3 mm

Commit message: did some stuff
Parts:
- removed JP1: Jumper_2_Open, TestPoint:TestPoint_2Pads_Pitch2.54mm_Drill0.8mm
- removed JP2: Jumper_2_Bridged, TestPoint:TestPoint_2Pads_Pitch2.54mm_Drill0.8mm
- removed U8: AW9523B, Package_DFN_QFN:QFN-24-1EP_4x4mm_P0.5mm_EP2.7x2.7mm
- added R12: 4.7k, Resistor_SMD:R_0603_1608Metric, F.Cu at (235.2, 46.4)
- added SW2: ~, ad-hoc:ALPSALPINE_TopPush_Button, F.Cu at (230.4, 49.6)
- added U10: SX1509, Package_DFN_QFN:QFN-28-1EP_4x4mm_P0.4mm_EP2.6x2.6mm, F.Cu at (220.4, 54.9)
- U6: value STZ12F405RGTx -> STM32F405RGTx
- moved R3 56.7 mm to (225.1, 53.8)
- moved R2 56.1 mm to (225.1, 55.4)
Connections:
- J1 pad 9: PB15 -> unconnected-(J1-Pin_9-Pad9)
- J2 pad 3: SCRN_SCL -> EXP_SCL
- J2 pad 4: SCRN_SDA -> EXP_SDA
- R2 pad 2: STEP_SCL -> EXP_SDA
- R3 pad 2: STEP_SDA -> EXP_SCL
- U2 pad 14: unconnected-(U2-MS2-Pad14) -> +3V3
- U4 pad 15: unconnected-(U4-MS1-Pad15) -> +3V3
- U5 pad 14: unconnected-(U5-MS2-Pad14) -> +3V3
- U5 pad 15: unconnected-(U5-MS1-Pad15) -> +3V3
- U6 pad 2: FAN1 -> DIAG_X1
- U6 pad 22: unconnected-(U6-PA6-Pad22) -> DIAG_Z1
- U6 pad 25: unconnected-(U6-PC5-Pad25) -> EN_Z1
- U6 pad 26: T0 -> DIAG_E1
- U6 pad 27: T1 -> DIR_E1
- U6 pad 28: T2 -> EN_E1
- U6 pad 29: STEP_SCL -> EXP_SCL
- U6 pad 3: FAN2 -> DIR_X1
- U6 pad 30: STEP_SDA -> EXP_SDA
- U6 pad 33: unconnected-(U6-PB12-Pad33) -> DIR_Z1
- U6 pad 36: PB15 -> INDEX_Z1
- U6 pad 4: FAN3 -> EN_X1
- U6 pad 56: unconnected-(U6-PB4-Pad56) -> STEP_Z1
- U6 pad 58: SCRN_SCL -> STEP_E1
- U6 pad 59: SCRN_SDA -> INDEX_E1
- U6 pad 61: unconnected-(U6-PB8-Pad61) -> STEP_X1
- U6 pad 62: unconnected-(U6-PB9-Pad62) -> INDEX_X1
Routing:
- net DIR_E1: track 108.4 -> 0.00 mm, vias 3 -> 0
- net EN_E1: track 94.7 -> 0.00 mm, vias 1 -> 0
- net DIAG_E1: track 87.8 -> 0.00 mm, vias 3 -> 0
- net STEP_E1: track 68.2 -> 0.00 mm, vias 1 -> 0
- net INDEX_E1: track 66.9 -> 0.00 mm, vias 2 -> 0
- net STEP_Z1: track 55.8 -> 0.00 mm, vias 1 -> 0
- net DIAG_Z1: track 49.0 -> 0.00 mm, vias 4 -> 0
- net SCRN_SCL: track 45.7 -> 0.00 mm, vias 6 -> 0
- net +3V3: track 272.2 -> 317.3 mm, vias 7 -> 10
- net EN_Z1: track 42.3 -> 0.00 mm, vias 1 -> 0
- net FAN1: track 40.9 -> 82.1 mm, vias 2 -> 6
- net SCRN_SDA: track 39.9 -> 0.00 mm, vias 4 -> 0
- net INDEX_Z1: track 37.3 -> 0.00 mm, vias 1 -> 0
- net FAN3: track 26.1 -> 62.7 mm, vias 4 -> 8
- net DIR_Z1: track 35.8 -> 0.00 mm, vias 1 -> 0
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